File: board/lenkungscontroller/lenkungscontroller.kicad_sch (KiCad schematic)
At the start: 34 parts, among them J1 Conn_01x03, J2 Conn_01x02_Female, J3 Conn_01x03, M1 Conn_01x02_Male, U1 TPS54360DDA, U3 A4950E, U8 SPX3819M5-L-3-3

Commit message: updated steering controller
Parts:
- removed ESP1: ESP32, luatos-footprint:Luatos, symbol project-parts:ESP32
- removed F1: Fuse, Fuse:Fuseholder_Cylinder-5x20mm_Stelvio-Kontek_PTF78_Horizontal_Open, symbol Device:Fuse
- added C2: 220uF, Capacitor_THT:CP_Radial_D10.0mm_P5.00mm, symbol Device:CP
- added D3: D, Diode_SMD:D_SOD-123F, symbol Device:D
- added R8: 1.5, Resistor_SMD:R_1210_3225Metric, symbol Device:R_US
- added U4: ESP32-C3_SUPERMINI, esp32c3supermini:MODULE_ESP32-C3_SUPERMINI, symbol ESP32-C3_SUPERMINI:ESP32-C3_SUPERMINI
- J2: footprint Connector_AMASS:AMASS_XT30UPB-M_1x02_P5.0mm_Vertical -> Connector_AMASS:AMASS_XT30PW-M_1x02_P2.50mm_Horizontal
- R6: value 0.25 -> 1.5
Connections:
- net 12V: now also D3.2 (A); no longer U8.1 (IN), U8.3 (EN)
- net 3_3V: now also U4.3.3 (3V3)
- net GND: now also C2.2, R8.2, U4.G (GND)
- net IN1: now also U4.7 (GPIO7)
- net IN2: now also U4.10 (GPIO10)
- net Poti: now also U4.5 (GPIO5)
- net Status: now also U4.6 (GPIO6)
- net VIN: now also J2.2 (Pin_2), C2.1
- net at R6.1, U3.7 (LSS): now also R8.1
- net Signal_In: now reaches J3.2 (Pin_2), R7.2
- net Signal_In: now also U4.4 (GPIO4)
- net Calibrate: now reaches Boot1.2, R5.2
- net Calibrate: now also U4.3 (GPIO3)
- new net: D3.1 (K), U8.1 (IN), U8.3 (EN)
- no-connect marks 8 -> 9
Other:
- moved on the sheet: C1, C4, C5, C6, C9, R3, Rvoltage_GND1
